File: sur2-adapter.kicad/sur2-adapter.kicad_pcb (KiCad board)
At the start: 2 copper layers, 9.5 x 14.5 mm, 3 parts, among them J1 Conn_SUR, J2 Conn_Pin, J3 Conn_PH

Commit message: Rev. 1.00 final version in production
Parts:
- moved J1 0.25 mm to (105.0, 112.5)
- moved J2 0.25 mm to (106.3, 104.6)
- moved J3 0.25 mm to (105.0, 105.3)
Other:
- board size 9.5 x 14.5 mm -> 10 x 14.5 mm
- board text added: "+"
- board text added: "-"
Changed lines of the file:
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@@
   (net 2 "GND")
   (footprint "user:JST_PH_S2B-PH-SM4-TB_1x02-1MP_P2.00mm_Horizontal" (layer "F.Cu")
-    (at 104.75 105.26 180)
+    (at 105 105.26 180)
     (descr "JST PH series connector, S2B-PH-SM4-TB (http://www.jst-mfg.com/product/pdf/eng/ePH.pdf), generated with kicad-footprint-generator")
     (tags "connector JST PH top entry")
+    (property "LCSC" "")
     (property "Sheetfile" "sur2-adapter.kicad_sch")
     (property "Sheetname" "")
+    (property "exclude_from_bom" "")
     (property "ki_description" "Generic connector, single row, 01x02, script generated (kicad-library-utils/schlib/autogen/connector/)")
     (property "ki_keywords" "connector")
-    (attr smd)
+    (attr smd exclude_from_pos_files exclude_from_bom)
     (fp_text reference "J3" (at 0 -5.8) (layer "F.SilkS") hide
         (effects (font (size 1 1) (thickness 0.15)))
@@
     (pad "2" smd roundrect (at 1 -2.85 180) (size 1 3.5) (layers "F.Cu" "F.Paste" "F.Mask") (roundrect_rratio 0.25)
       (net 2 "GND") (pinfunction "Pin_2") (pintype "passive"))
-    (pad "MP" smd roundrect (at -3.35 2.9 180) (size 1.5 3.4) (layers "F.Cu" "F.Paste" "F.Mask") (roundrect_rratio 0.166667))
-    (pad "MP" smd roundrect (at 3.35 2.9 180) (size 1.5 3.4) (layers "F.Cu" "F.Paste" "F.Mask") (roundrect_rratio 0.166667))
+    (pad "MP" smd roundrect (at -3.35 2.9 180) (size 1.5 3.4) (layers "F.Cu" "F.Paste" "F.Mask") (roundrect_rratio 0.1666673333))
+    (pad "MP" smd roundrect (at 3.35 2.9 180) (size 1.5 3.4) (layers "F.Cu" "F.Paste" "F.Mask") (roundrect_rratio 0.1666673333))
     (model "${KICAD6_3DMODEL_DIR}/Connector_JST.3dshapes/JST_PH_S2B-PH-SM4-TB_1x02-1MP_P2.00mm_Horizontal.wrl"
       (offset (xyz 0 0 0))
@@
   )
   (footprint "Connector_JST:JST_SUR_BM02B-SURS-TF_1x02-1MP_P0.80mm_Vertical" (layer "F.Cu")
-    (at 104.75 112.45 180)
+    (at 105 112.45 180)
     (descr "JST SUR series connector, BM02B-SURS-TF (http://www.jst-mfg.com/product/pdf/eng/eSUR.pdf), generated with kicad-footprint-generator")
     (tags "connector JST SUR side entry")
+    (property "LCSC" "C385130")
     (property "Sheetfile" "sur2-adapter.kicad_sch")
     (property "Sheetname" "")
@@
     (pad "2" smd roundrect (at 0.4 0.85 180) (size 0.5 1.1) (layers "F.Cu" "F.Paste" "F.Mask") (roundrect_rratio 0.25)
       (net 2 "GND") (pinfunction "Pin_2") (pintype "passive"))
-    (pad "MP" smd roundrect (at -1.7 -0.55 180) (size 1.2 1.7) (layers "F.Cu" "F.Paste" "F.Mask") (roundrect_rratio 0.208333))
-    (pad "MP" smd roundrect (at 1.7 -0.55 180) (size 1.2 1.7) (layers "F.Cu" "F.Paste" "F.Mask") (roundrect_rratio 0.208333))
+    (pad "MP" smd roundrect (at -1.7 -0.55 180) (size 1.2 1.7) (layers "F.Cu" "F.Paste" "F.Mask") (roundrect_rratio 0.2083333333))
+    (pad "MP" smd roundrect (at 1.7 -0.55 180) (size 1.2 1.7) (layers "F.Cu" "F.Paste" "F.Mask") (roundrect_rratio 0.2083333333))
     (model "${KICAD6_3DMODEL_DIR}/Connector_JST.3dshapes/JST_SUR_BM02B-SURS-TF_1x02-1MP_P0.80mm_Vertical.wrl"
       (offset (xyz 0 0 0))
@@
   )
   (footprint "Connector_PinHeader_2.54mm:PinHeader_1x02_P2.54mm_Vertical" (layer "B.Cu")
-    (at 106.025 104.6 90)
+    (at 106.275 104.6 90)
     (descr "Through hole straight pin header, 1x02, 2.54mm pitch, single row")
     (tags "Through hole pin header THT 1x02 2.54mm single row")
+    (property "LCSC" "")
     (property "Sheetfile" "sur2-adapter.kicad_sch")
     (property "Sheetname" "")
+    (property "exclude_from_bom" "")
     (property "ki_description" "Generic connector, single row, 01x02, script generated (kicad-library-utils/schlib/autogen/connector/)")
     (property "ki_keywords" "connector")
-    (attr through_hole)
+    (attr through_hole exclude_from_pos_files exclude_from_bom)
     (fp_text reference "J2" (at 0 2.33 90) (layer "B.SilkS") hide
         (effects (font (size 1 1) (thickness 0.15)) (justify mirror))
@@
     )
   )
-  (gr_rect (start 100 100) (end 109.5 114.5)
+  (gr_rect (start 100 100) (end 110 114.5)
     (stroke (width 0.05) (type default)) (fill none) (layer "Edge.Cuts"))
-  (gr_text "Rev. 1.00" (at 107.8 114.3 -90) (layer "B.SilkS")
+  (gr_text "Rev. 1.00" (at 108.05 114.3 -90) (layer "B.SilkS")
     (effects (font (size 1 1) (thickness 0.1)) (justify left bottom mirror))
   )
-  (via (at 108.3 109.2) (size 0.6) (drill 0.3) (layers "F.Cu" "B.Cu") (free) (net 1))
-  (via (at 101.2 109.2) (size 0.6) (drill 0.3) (layers "F.Cu" "B.Cu") (free) (net 2))
+  (gr_text "+" (at 106.76 109.86) (layer "F.SilkS")
+    (effects (font (size 1 1) (thickness 0.1)) (justify left bottom))
+  )
+  (gr_text "-" (at 103 103.1) (layer "F.SilkS")
+    (effects (font (size 1 1) (thickness 0.1)) (justify left bottom))
+  )
+  (gr_text "-" (at 101.75 109.8) (layer "F.SilkS")
+    (effects (font (size 1 1) (thickness 0.1)) (justify left bottom))
+  )
+  (gr_text "+" (at 105.6 103.15) (layer "F.SilkS")
+    (effects (font (size 1 1) (thickness 0.1)) (justify left bottom))
+  )
+  (gr_text "-" (at 100.7 112.05) (layer "F.SilkS")
+    (effects (font (size 1 1) (thickness 0.1)) (justify left bottom))
+  )
+  (gr_text "+" (at 107.85 112) (layer "F.SilkS")
+    (effects (font (size 1 1) (thickness 0.1)) (justify left bottom))
+  )
+  (via (at 108.55 109.2) (size 0.6) (drill 0.3) (layers "F.Cu" "B.Cu") (free) (net 1))
+  (via (at 101.45 109.2) (size 0.6) (drill 0.3) (layers "F.Cu" "B.Cu") (free) (net 2))
   (zone (net 2) (net_name "GND") (layers "F&B.Cu") (name "GND") (hatch edge 0.5)
     (connect_pads (clearance 0))
@@
     (polygon
       (pts
-        (xy 99.7 99.6)
-        (xy 104.7 99.6)
-        (xy 104.7 114.8)
-        (xy 99.8 114.8)
+        (xy 99.95 99.6)
+        (xy 104.95 99.6)
+        (xy 104.95 114.8)
+        (xy 100.05 114.8)
       )
     )
@@
     (polygon
       (pts
-        (xy 104.8 99.6)
-        (xy 109.7 99.6)
-        (xy 109.7 114.8)
-        (xy 104.9 114.8)
+        (xy 105.05 99.6)
+        (xy 109.95 99.6)
+        (xy 109.95 114.8)
+        (xy 105.15 114.8)
       )
     )
