File: sur2-adapter.kicad/sur2-adapter.kicad_sch (KiCad schematic)
At the start: 3 parts, among them J1 Conn_SUR, J2 Conn_Pin, J3 Conn_PH

Commit message: Rev. 1.00 final version in production
Parts:
- J1: LCSC (none) -> C385130
- J2, J3: now left out of the parts list
Changed lines of the file:
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@@
+      (effects (font (size 1.27 1.27)) hide)
+    )
+    (property "LCSC" "C385130" (at 97.79 59.69 0)
       (effects (font (size 1.27 1.27)) hide)
     )
@@
   )
   (symbol (lib_id "Connector_Generic:Conn_01x02") (at 97.79 73.66 0) (unit 1)
-    (in_bom yes) (on_board yes) (dnp no) (fields_autoplaced)
+    (in_bom no) (on_board yes) (dnp no) (fields_autoplaced)
     (property "Reference" "J2" (at 100.33 73.66 0)
       (effects (font (size 1.27 1.27)) (justify left))
@@
       (effects (font (size 1.27 1.27)) hide)
     )
+    (property "LCSC" "" (at 97.79 73.66 0)
+      (effects (font (size 1.27 1.27)))
+    )
     (pin "2")
     (pin "1")
@@
   )
   (symbol (lib_id "Connector_Generic:Conn_01x02") (at 97.79 86.36 0) (unit 1)
-    (in_bom yes) (on_board yes) (dnp no) (fields_autoplaced)
+    (in_bom no) (on_board yes) (dnp no) (fields_autoplaced)
     (property "Reference" "J3" (at 100.33 86.36 0)
       (effects (font (size 1.27 1.27)) (justify left))
@@
       (effects (font (size 1.27 1.27)) hide)
     )
+    (property "LCSC" "" (at 97.79 86.36 0)
+      (effects (font (size 1.27 1.27)))
+    )
     (pin "2")
